File: mangoh-red.sch (KiCad schematic (older format))
At the start: 0 parts

Commit message: Updating
Changed lines of the file:
@@
 EESchema Schematic File Version 4
+LIBS:mangoh-red-cache
 EELAYER 26 0
 EELAYER END
@@
 $EndDescr
 $Sheet
-S 10150 1550 3650 400
+S 10200 1500 3650 400
 U 5B20369B
 F0 "2. CF3 Socket" 128
