File: mangoh-red.kicad_pcb (KiCad board)
At the start: 6 copper layers, 70 x 61.8 mm, 570 parts, among them CN1000 uFL, CN301 uFL, CN302 uFL, CN303 uFL, CN304 USB_A, CN305 USB_B_Micro, CN306 Conn_02x19_Counter_Clockwise, CN307 Conn_02x13_Odd_Even, CN310 Conn_02x03_Odd_Even, CN312 Conn_02x03_Odd_Even, CN500 JP036-RT3B4AB, CN801 USB_B_Micro, CN802 Conn_01x02, CN804 Conn_01x03, J200 CF3-Socket, Q312 NSBC114YDP6T5G, Q400 NSBC114YDP6T5G, Q405 NSBC114YDP6T5G, Q600 PDTC115EM, SW401 Conn_02x08_Counter_Clockwise, U1000 MT7697, U1001 MX25L3233FM1I-08G_TR, U1004 SX1509BIULTRT, U1005 TPS61253YFFR, U1006 CP2130-F01-GM, U1007 24AA32AF-I-MNY, U1010 74LVC2G126HD4-7, U1020 74LVC2G126HD4-7, U301 FT230XQ-R, U302 TS3A5018RSVR, U304 74LVC2G126HD4-7, U306 FXMA108BQX, U307 FXMA108BQX, U337 FXMA108BQX, U400 NCP303LSN30T1G, U401 74AUP1G08GM, U402 74AUP1G08GM, U404 TCA9546APWR, U405 74AUP1G08GM, U500 WM8944BECS_R, U501 TS3A5018RSVR, U600 XC6223H29B9R-G, U610 TXS02612ZQSR, U701 USB3503A-1-GL-TR, U702 MIC2026-1YM, U704 BMI160, U705 BMP280, U706 PNJ4K01F, U800 BQ24296RGER, U801 LTC2942IDCB_TRMPBF, U900 TPS7A7300, U901 TPS62420DRC, U903 XC6221A182MR, Y1000 CT2520DB26000C0FZZA1

Commit message: Update
Parts:
- added CN1: Conn_02x05_Odd_Even, Connector_PinSocket_1.27mm:PinSocket_2x05_P1.27mm_Vertical, F.Cu at (183.7, 44.9)
- added CN401: Conn_02x05_Odd_Even, Connector_PinSocket_1.27mm:PinSocket_2x05_P1.27mm_Vertical, F.Cu at (188.8, 44.9)
- added D200: LED_PAD (1204), LED_SMD:LED_1206_3216Metric, F.Cu at (194.3, 57.1)
- added D305: TPD4S012DRYR, Package_SON:WSON-6_1.5x1.5mm_P0.5mm, F.Cu at (201.6, 44.8)
- added D401: LED_PAD (1204), LED_SMD:LED_1206_3216Metric, F.Cu at (193.6, 44.9)
- added D402: LED_PAD (1204), LED_SMD:LED_1206_3216Metric, F.Cu at (193.6, 48.3)
- added D600: RCLAMP0503N, Package_SON:WSON-6_1.5x1.5mm_P0.5mm, F.Cu at (185.6, 57.0)
- added D601: TPD6E004RSER, Package_DFN_QFN:UDFN-10_1.35x2.6mm_P0.5mm, F.Cu at (182.2, 57.5)
- added D800: TPD4S012DRYR, Package_SON:WSON-6_1.5x1.5mm_P0.5mm, F.Cu at (202.6, 52.1)
- added R301: 10k, Capacitor_SMD:C_0402_1005Metric, F.Cu at (204.8, 44.2)
- added R349: 820k, Capacitor_SMD:C_0402_1005Metric, F.Cu at (204.8, 46.2)
- D301, D302, D303, D400: footprint LEDs:LED_0402 -> LED_SMD:LED_0402_1005Metric
- D410, D801, D803: footprint LEDs:LED_0603 -> LED_SMD:LED_0603_1608Metric
- R822, R901: footprint Resistor_SMD:R_0402_1005Metric -> Capacitor_SMD:C_0402_1005Metric
Connections:
- CN801 pad 2: (no net) -> Net-(CN801-Pad2)
- CN801 pad 3: (no net) -> Net-(CN801-Pad3)
- J200 pad 106: (no net) -> Net-(D200-Pad1)
- J200 pad 27: (no net) -> UIM1_CLK
- J200 pad 29: (no net) -> UIM1_RESET
- Q400 pad 3: (no net) -> Net-(D402-Pad1)
- Q400 pad 6: (no net) -> Net-(D401-Pad1)
- R222 pad 2: (no net) -> Net-(D200-Pad2)
- R413 pad 1: (no net) -> Net-(D401-Pad2)
- R435 pad 1: (no net) -> Net-(D402-Pad2)

Commit message: Update
Parts:
- C1017: footprint Capacitor_SMD:C_0402_1005Metric -> Capacitor_SMD:C_0603_1608Metric
- C1100: footprint Capacitor_SMD:C_0201_0603Metric -> Capacitor_SMD:C_0402_1005Metric
- C812: footprint Capacitor_SMD:C_0402_1005Metric -> Capacitor_SMD:C_1206_3216Metric
- CN1, CN401: footprint Connector_PinSocket_1.27mm:PinSocket_2x05_P1.27mm_Vertical -> Connector_PinSocket_1.27mm:PinSocket_2x05_P1.27mm_Vertical_SMD
- R301, R349, R822, R901: footprint Capacitor_SMD:C_0402_1005Metric -> Resistor_SMD:R_0402_1005Metric
- moved CN1 46.9 mm to (167.0, 88.7)
- moved CN401 46.4 mm to (177.0, 89.7)
- moved D600 7.54 mm to (179.0, 60.7)
- moved D601 3.25 mm to (179.0, 56.7)

Commit message: Update
Parts:
- added ANT1000: WLA.01, MangOH-Red:WLA.01, F.Cu at (210.8, 49.5)
- added L800: TCM1210-900-2P-T000, MangOH-Red:EXC24C, F.Cu at (228.8, 47.9)
- added L801: 3.3u, MangOH-Red:IND_2P_0400x0400_0237CC_COILCRAFT, F.Cu at (224.3, 48.7)
- C922: footprint Capacitor_SMD:C_0402_1005Metric -> MangOH-Red:CAP_2P_0720x0630_POL_NIB
- D200, D401, D402: value LED_PAD (1204) -> LED_PAD; footprint LED_SMD:LED_1206_3216Metric -> MangOH-Red:12-21SYGC_S530-E2_TR8
- D305, D600, D800: footprint Package_SON:WSON-6_1.5x1.5mm_P0.5mm -> MangOH-Red:DFN_6P_0145x0100_0050CC
- D601: footprint Package_DFN_QFN:UDFN-10_1.35x2.6mm_P0.5mm -> MangOH-Red:QFN_8P_0150x0150_0050CC
- U302, U501: footprint MangOH-Red:QFN_14P_0250x0300_0050CC -> MangOH-Red:QFN_16P_0260x0180_0040CC
- U401, U402, U405: footprint Package_DFN_QFN:DFN-6-1EP_2x2mm_P0.5mm_EP0.61x1.42mm -> MangOH-Red:DFN_6P_0145x0100_0050CC
- U706: footprint Package_DFN_QFN:DFN-6-1EP_2x2mm_P0.5mm_EP0.61x1.42mm -> MangOH-Red:DFN_6P_0155x0150_0050CC
Connections:
- D600 pad 1: UIM1_RESET -> (no net)
- D600 pad 3: UIM1_CLK -> (no net)
- D600 pad 4: UIM1_DATA -> (no net)
- D600 pad 5: VCC -> (no net)
- D600 pad 6: GND -> (no net)
- J200 pad 12: (no net) -> USB_D-
- J200 pad 13: (no net) -> USB_D+
- J200 pad 27: UIM1_CLK -> (no net)
- J200 pad 29: UIM1_RESET -> (no net)
